Commit message: constant joint state pubs

File: ar3/ar3.urdf (robot description, URDF)
Before this commit: robot ar3, 7 links, 6 joints
Joints:
- joint joint_4: origin xyz=0 0 0.00675 rpy=1.5708 -1.2554 -1.5708 -> xyz=0 0 0.00675 rpy=1.5708 -1.2554 -1.05

Commit message: smoother operation

File: ar3/ar3.urdf (robot description, URDF)
Before this commit: robot ar3, 7 links, 6 joints
Joints:
- joint joint_5: axis -1 0 0 -> 1 0 0

Commit message: added joint control mode

File: ar3/ar3.urdf (robot description, URDF)
Before this commit: robot ar3, 7 links, 6 joints
Joints:
- joint joint_5: origin xyz=0 0 -0.22225 rpy=3.1416 0 -2.8262 -> xyz=0 0 -0.22225 rpy=4.05 0 -2.8262
